Commit message: fix(urdf): kamera açısı 30°'den 6°'ye düşürüldü
Zemine daha sığ bakış açısı için cam_pitch 0.523'ten 0.1 rad'a güncellendi.

Co-Authored-By: Claude Sonnet 4.6 <noreply@anthropic.com>

File: src/aircraft_taxi_description/urdf/aircraft_taxi.urdf.xacro (robot description, xacro)
@@ -27,8 +27,8 @@
   <xacro:property name="caster_x"      value="1.1"/>
   <xacro:property name="caster_radius" value="0.12"/>
-  <!-- Kamera konumu (gövde ön-altı, zemine ~30° bakış) -->
+  <!-- Kamera konumu (gövde ön-altı, zemine ~6° bakış) -->
   <xacro:property name="cam_x"    value="1.3"/>
   <xacro:property name="cam_z"    value="-0.15"/>
-  <xacro:property name="cam_pitch" value="0.523"/>   <!-- ~30 derece -->
+  <xacro:property name="cam_pitch" value="0.1"/>     <!-- ~6 derece -->
   <!-- Lidar konumu (gövde ön-üstü) -->
   <xacro:property name="lidar_x"  value="1.1"/>
